Commit message: carebuddy_urdf

File: carebuddy_description/urdf/carebuddy.xacro (robot description, xacro)
@@ -1,6 +1,6 @@
 <?xml version="1.0" encoding="utf-8"?>
-<robot name="proj7" xmlns:xacro="http://www.ros.org/wiki/xacro">
-<xacro:include filename="$(find proj7)/urdf/gazebo_refs_xArm.xacro" />
-<xacro:include filename="$(find proj7)/urdf/transmission_xArm.xacro" />
+<robot name="carebuddy_description" xmlns:xacro="http://www.ros.org/wiki/xacro">
+<xacro:include filename="$(find carebuddy_description)/urdf/gazebo_refs_xArm.xacro" />
+<xacro:include filename="$(find carebuddy_description)/urdf/transmission_xArm.xacro" />
 <link name="base_link">
     <inertial>
@@ -12,5 +12,5 @@
       <origin xyz="0 0 0" rpy="0 0 0"/>
       <geometry>
-        <mesh filename="package://proj7/meshes/base_link.STL" scale="0.5 0.5 0.5"/>
+        <mesh filename="package://carebuddy_description/meshes/base_link.STL" scale="0.5 0.5 0.5"/>
       </geometry>
       <material name="">
@@ -21,5 +21,5 @@
       <origin xyz="0 0 0" rpy="0 0 0"/>
       <geometry>
-        <mesh filename="package://proj7/meshes/base_link.STL" scale="0.5 0.5 0.5"/>
+        <mesh filename="package://carebuddy_description/meshes/base_link.STL" scale="0.5 0.5 0.5"/>
       </geometry>
     </collision>
@@ -34,5 +34,5 @@
       <origin xyz="0.0 0 0" rpy="0 0 0"/>
       <geometry>
-        <mesh filename="package://proj7/meshes/wheel1.STL" scale="0.5 0.5 0.5"/>
+        <mesh filename="package://carebuddy_description/meshes/wheel1.STL" scale="0.5 0.5 0.5"/>
       </geometry>
       <material name="">
@@ -43,5 +43,5 @@
       <origin xyz="0 0 0" rpy="0 0 0"/>
       <geometry>
-        <mesh filename="package://proj7/meshes/wheel1.STL" scale="0.5 0.5 0.5"/>
+        <mesh filename="package://carebuddy_description/meshes/wheel1.STL" scale="0.5 0.5 0.5"/>
       </geometry>
     </collision>
@@ -62,5 +62,5 @@
       <origin xyz="0 0 0" rpy="0 0 0"/>
       <geometry>
-        <mesh filename="package://proj7/meshes/wheel2.STL" scale="0.5 0.5 0.5"/>
+        <mesh filename="package://carebuddy_description/meshes/wheel2.STL" scale="0.5 0.5 0.5"/>
       </geometry>
     </visual>
@@ -68,5 +68,5 @@
       <origin xyz="0 0 0" rpy="0 0 0"/>
       <geometry>
-        <mesh filename="package://proj7/meshes/wheel2.STL" scale="0.5 0.5 0.5"/>
+        <mesh filename="package://carebuddy_description/meshes/wheel2.STL" scale="0.5 0.5 0.5"/>
       </geometry>
     </collision>
@@ -87,5 +87,5 @@
       <origin xyz="0 0 0" rpy="0 0 0"/>
       <geometry>
-        <mesh filename="package://proj7/meshes/wheel3.STL" scale="0.5 0.5 0.5"/>
+        <mesh filename="package://carebuddy_description/meshes/wheel3.STL" scale="0.5 0.5 0.5"/>
       </geometry>
       <material name="">
@@ -96,5 +96,5 @@
       <origin xyz="0 0 0" rpy="0 0 0"/>
       <geometry>
-        <mesh filename="package://proj7/meshes/wheel3.STL" scale="0.5 0.5 0.5"/>
+        <mesh filename="package://carebuddy_description/meshes/wheel3.STL" scale="0.5 0.5 0.5"/>
       </geometry>
     </collision>
@@ -115,5 +115,5 @@
       <origin xyz="0 0 0" rpy="0 0 0"/>
       <geometry>
-        <mesh filename="package://proj7/meshes/wheel4.STL" scale="0.5 0.5 0.5" />
+        <mesh filename="package://carebuddy_description/meshes/wheel4.STL" scale="0.5 0.5 0.5" />
       </geometry>
     </visual>
@@ -121,5 +121,5 @@
       <origin xyz="0 0 0" rpy="0 0 0"/>
       <geometry>
-        <mesh filename="package://proj7/meshes/wheel4.STL" scale="0.5 0.5 0.5" />
+        <mesh filename="package://carebuddy_description/meshes/wheel4.STL" scale="0.5 0.5 0.5" />
       </geometry>
     </collision>

File: carebuddy_description/urdf/gazebo_refs_xArm.xacro (robot description, xacro)
@@ -1,3 +1,3 @@
-<robot name="proj7" xmlns:xacro="http://www.ros.org/wiki/xacro" >
+<robot name="carebuddy" xmlns:xacro="http://www.ros.org/wiki/xacro" >
 <xacro:macro name="Colors" params="wheel ">
     <gazebo reference="${wheel}">

File: carebuddy_description/urdf/transmission.trans.xacro (robot description, xacro)
@@ -1,3 +1,3 @@
-<robot name="proj7" xmlns:xacro="http://www.ros.org/wiki/xacro">
+<robot name="carebuddy" xmlns:xacro="http://www.ros.org/wiki/xacro">
 <!-- Joints -->
 <xacro:macro name="Transmission_Block" params="prefix suffix">

File: carebuddy_description/urdf/transmission_xArm.xacro (robot description, xacro)
@@ -1,3 +1,3 @@
-<robot name="proj7" xmlns:xacro="http://www.ros.org/wiki/xacro">
+<robot name="carebuddy" xmlns:xacro="http://www.ros.org/wiki/xacro">
 <!-- Joints -->
 <xacro:macro name="Transmission_Block" params="prefix suffix">
